File: hardware/lyrebird-dac-reva/lyrebird-dac.kicad_sch (KiCad schematic)
At the start: 42 parts, among them J1 Mezzanine 2x40, U1 clock divider /2, U2 74AVC4T245, U3a 16-bit register (ch L) PLACEH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, U3b 16-bit register (ch L) PLACEH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, U4a 16-bit register (ch R) PLACEH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, U4b 16-bit register (ch R) PLACEH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, U5 LT3045 element reference, U6 LT3045 clock chain, U7 output op amp PLACEHOLDER, U8 LT3094 op amp negative rail, U9 LT3045 header-side 2.5 V, Y1 CCHD-957 49.152MHz, Y2 CCHD-957 45.1584MHz

Commit message: Draw wires in the schematics instead of relying on net labels
Labels alone are hard to follow, so nets of two or three pins are now drawn
as wires and the parts sharing one are placed next to each other to keep the
wire short. That covers 119 of the main board's 125 nets and 68 of the
module's 82.

The split follows what a person does by hand rather than a rule of thumb.
Ground, the supply rails and the element bus stay as labels, because a wire
joining 245 ground pins is not a drawing anyone can read. Everything else is
a line you can trace.

Parts are clustered by the nets that join them, 94 clusters on the main board
and 19 on the module, so a wire is usually a short hop between neighbours
rather than a line across the sheet. Two-pin nets route as an L, three-pin
nets as a comb to a shared vertical. There is still no global routing, which
is the part that cannot be automated.

One bug had been silently eating most of the connectivity. KiCad symbols may
inherit from a base through `extends`, carrying its graphics and pins while
overriding properties. The reader took such a symbol at face value and saw no
pins at all, so 58 of 68 candidate nets on the module failed their pin lookup
and went unwired. Inheritance is now flattened before pins are read.

PDFs of both schematics are committed beside their boards.

Co-Authored-By: Claude Opus 5 <noreply@anthropic.com>
Connections:
- net +3V3_CLK is gone; now on net +2V5: U2.16 (VCCB), U6.10 (OUT), U6.9 (OUTS), Y1.4 (Vdd), Y2.4 (Vdd)
- net +3V3_REF is gone; now on net +2V5: U5.10 (OUT), U5.9 (OUTS)
- net +5V is gone; now on net +2V5: J1.71 (Pin_71), J1.73 (Pin_73), J1.75 (Pin_75), J1.77 (Pin_77), J1.79 (Pin_79), U5.1 (IN), U5.2 (IN), U5.3 (EN/UV), U5.6 (PGFB), U6.1 (IN), U6.2 (IN), U6.3 (EN/UV), U6.6 (PGFB), U9.1 (IN), U9.2 (IN), U9.3 (EN/UV), U9.6 (PGFB)
- net ELEM0 is gone; now on net ELEM28: J1.1 (Pin_1)
- net ELEM1 is gone; now on net ELEM28: J1.3 (Pin_3)
- net ELEM10 is gone; now on net ELEM28: J1.21 (Pin_21)
- net ELEM11 is gone; now on net ELEM28: J1.23 (Pin_23)
- net ELEM12 is gone; now on net ELEM28: J1.25 (Pin_25)
- net ELEM13 is gone; now on net ELEM28: J1.27 (Pin_27)
- net ELEM14 is gone; now on net ELEM28: J1.29 (Pin_29)
- net ELEM15 is gone; now on net ELEM28: J1.31 (Pin_31)
- net ELEM16 is gone; now on net ELEM28: J1.33 (Pin_33)
- net ELEM17 is gone; now on net ELEM28: J1.35 (Pin_35)
- net ELEM18 is gone; now on net ELEM28: J1.37 (Pin_37)
- net ELEM19 is gone; now on net ELEM28: J1.39 (Pin_39)
- net ELEM2 is gone; now on net ELEM28: J1.5 (Pin_5)
- net ELEM20 is gone; now on net ELEM28: J1.41 (Pin_41)
- net ELEM21 is gone; now on net ELEM28: J1.43 (Pin_43)
- net ELEM22 is gone; now on net ELEM28: J1.45 (Pin_45)
- net ELEM23 is gone; now on net ELEM28: J1.47 (Pin_47)
- net ELEM24 is gone; now on net ELEM28: J1.49 (Pin_49)
- net ELEM25 is gone; now on net ELEM28: J1.51 (Pin_51)
- net ELEM26 is gone; now on net ELEM28: J1.53 (Pin_53)
- net ELEM27 is gone; now on net ELEM28: J1.55 (Pin_55)
- net ELEM29 is gone; now on net ELEM28: J1.59 (Pin_59)
- net ELEM3 is gone; now on net ELEM28: J1.7 (Pin_7)
- net ELEM30 is gone; now on net ELEM28: J1.61 (Pin_61)
- net ELEM31 is gone; now on net ELEM28: J1.63 (Pin_63)
- net ELEM4 is gone; now on net ELEM28: J1.9 (Pin_9)
- net ELEM5 is gone; now on net ELEM28: J1.11 (Pin_11)
- net ELEM6 is gone; now on net ELEM28: J1.13 (Pin_13)
- net ELEM7 is gone; now on net ELEM28: J1.15 (Pin_15)
- net ELEM8 is gone; now on net ELEM28: J1.17 (Pin_17)
- net ELEM9 is gone; now on net ELEM28: J1.19 (Pin_19)
- net GND is gone; now on net ELEM28: J1.10 (Pin_10), J1.12 (Pin_12), J1.14 (Pin_14), J1.16 (Pin_16), J1.18 (Pin_18), J1.2 (Pin_2), J1.20 (Pin_20), J1.22 (Pin_22), J1.24 (Pin_24), J1.26 (Pin_26), J1.28 (Pin_28), J1.30 (Pin_30), J1.32 (Pin_32), J1.34 (Pin_34), J1.36 (Pin_36), J1.38 (Pin_38), J1.4 (Pin_4), J1.40 (Pin_40), J1.42 (Pin_42), J1.44 (Pin_44), J1.46 (Pin_46), J1.48 (Pin_48), J1.50 (Pin_50), J1.52 (Pin_52), J1.54 (Pin_54), J1.56 (Pin_56), J1.58 (Pin_58), J1.6 (Pin_6), J1.60 (Pin_60), J1.62 (Pin_62), J1.64 (Pin_64), J1.72 (Pin_72), J1.74 (Pin_74), J1.76 (Pin_76), J1.78 (Pin_78), J1.8 (Pin_8), J1.80 (Pin_80), U2.12 (1B2), U2.14 (2~{OE}), U2.15 (1~{OE}), U2.2 (1DIR), U2.8 (GND), U2.9 (GND), U5.11 (GND), U5.5 (ILIM), U5.8 (GND), U6.11 (GND), U6.5 (ILIM), U6.8 (GND), U9.11 (GND), U9.5 (ILIM), U9.8 (GND), Y1.2 (GND), Y2.2 (GND)
- net ID0 is gone; now on net ELEM28: J1.69 (Pin_69)
- net ID1 is gone; now on net ELEM28: J1.70 (Pin_70)
- net MCLK is gone; now on net ELEM28: J1.65 (Pin_65), U2.4 (1A1)
- net MUTE_N is gone; now on net ELEM28: J1.68 (Pin_68)
- net N$10 is gone; now on net ELEM28: RN3.2 (R2.1)
- net N$11 is gone; now on net ELEM28: RN3.3 (R3.1)
- net N$12 is gone; now on net ELEM28: RN3.4 (R4.1)
- net N$13 is gone; now on net ELEM28: RN4.1 (R1.1)
- net N$14 is gone; now on net ELEM28: RN4.2 (R2.1)
- net N$16 is gone; now on net ELEM28: RN4.4 (R4.1)
- net N$17 is gone; now on net ELEM28: RN5.1 (R1.1)
- net N$18 is gone; now on net ELEM28: RN5.2 (R2.1)
- net N$19 is gone; now on net ELEM28: RN5.3 (R3.1)
- net N$2 is gone; now on net ELEM28: RN1.2 (R2.1)
- net N$20 is gone; now on net ELEM28: RN5.4 (R4.1)
- net N$21 is gone; now on net ELEM28: RN6.1 (R1.1)
- net N$23 is gone; now on net ELEM28: RN6.3 (R3.1)
- net N$24 is gone; now on net ELEM28: RN6.4 (R4.1)
- net N$25 is gone; now on net ELEM28: RN7.1 (R1.1)
- net N$26 is gone; now on net ELEM28: RN7.2 (R2.1)
- net N$27 is gone; now on net ELEM28: RN7.3 (R3.1)
- net N$28 is gone; now on net ELEM28: RN7.4 (R4.1)
- net N$29 is gone; now on net +2V5: U5.7 (SET)
- net N$30 is gone; now on net +2V5: U6.7 (SET)
- net N$31 is gone; now on net +2V5: U9.7 (SET)
- net N$5 is gone; now on net ELEM28: RN2.1 (R1.1)
- net N$6 is gone; now on net ELEM28: RN2.2 (R2.1)
- net N$7 is gone; now on net ELEM28: RN2.3 (R3.1)
- net N$9 is gone; now on net ELEM28: RN3.1 (R1.1)
- net OSC_EN_441 is gone; now on net ELEM28: J1.66 (Pin_66), U2.7 (2A2)
- net OSC_EN_441_3V3 is gone; now on net ELEM28: U2.10 (2B2), Y2.1 (EN)
- net OSC_EN_48 is gone; now on net ELEM28: J1.67 (Pin_67), U2.6 (2A1)
- net OSC_EN_48_3V3 is gone; now on net ELEM28: U2.11 (2B1), Y1.1 (EN)
- net OSC_RAW is gone; now on net ELEM28: Y1.3 (OUT), Y2.3 (OUT)
- net SUM_N is gone; now on net ELEM28: RN2.5 (R4.2), RN3.5 (R4.2), RN3.6 (R3.2), RN3.7 (R2.2), RN3.8 (R1.2), RN4.7 (R2.2), RN4.8 (R1.2), RN6.5 (R4.2), RN6.6 (R3.2), RN6.7 (R2.2), RN7.5 (R4.2), RN7.6 (R3.2), RN7.7 (R2.2), RN7.8 (R1.2)
- net SUM_P is gone; now on net ELEM28: RN1.5 (R4.2), RN1.6 (R3.2), RN1.7 (R2.2), RN1.8 (R1.2), RN2.6 (R3.2), RN2.7 (R2.2), RN2.8 (R1.2), RN4.5 (R4.2), RN4.6 (R3.2), RN5.5 (R4.2), RN5.6 (R3.2), RN5.7 (R2.2), RN5.8 (R1.2), RN6.8 (R1.2)
- net +2V5: now also U1.8 (VCC), U3a.20 (VCC), U3b.20 (VCC), U4a.20 (VCC), U4b.20 (VCC)
- net ELEM28: now also U1.1 (C), U1.4 (GND), U3a.1 (OE), U3a.10 (GND), U3a.13 (Q6), U3a.16 (Q3), U3a.17 (Q2), U3a.18 (Q1), U3a.2 (D0), U3a.3 (D1), U3a.4 (D2), U3a.5 (D3), U3a.6 (D4), U3a.7 (D5), U3a.8 (D6), U3b.1 (OE), U3b.10 (GND), U3b.13 (Q6), U3b.14 (Q5), U3b.15 (Q4), U3b.16 (Q3), U3b.17 (Q2), U3b.18 (Q1), U3b.2 (D0), U3b.3 (D1), U3b.4 (D2), U3b.5 (D3), U3b.6 (D4), U3b.7 (D5), U3b.8 (D6), U4a.1 (OE), U4a.10 (GND), U4a.13 (Q6), U4a.14 (Q5), U4a.15 (Q4), U4a.16 (Q3), U4a.17 (Q2), U4a.18 (Q1), U4a.2 (D0), U4a.3 (D1), U4a.4 (D2), U4a.5 (D3), U4a.6 (D4), U4a.7 (D5), U4a.8 (D6), U4b.1 (OE), U4b.10 (GND), U4b.13 (Q6), U4b.14 (Q5), U4b.15 (Q4), U4b.16 (Q3), U4b.17 (Q2), U4b.18 (Q1), U4b.2 (D0), U4b.3 (D1), U4b.4 (D2), U4b.5 (D3), U4b.6 (D4), U4b.7 (D5), U4b.8 (D6), U8.9 (GND)
- net ELEM_CLK: no longer names the net of U2.13 (1B1)
- net ELEM_CLK: now also U1.5 (Q)
- net N$1: no longer names the net of RN1.1 (R1.1)
- net N$1: now also U3a.12 (Q7)
- net N$15: no longer names the net of RN4.3 (R3.1)
- net N$15: now also U4a.12 (Q7)
- net N$22: no longer names the net of RN6.2 (R2.1)
- net N$22: now also U4b.12 (Q7)
- net N$3: no longer names the net of RN1.3 (R3.1)
- net N$3: now also U3a.14 (Q5)
- net N$4: no longer names the net of RN1.4 (R4.1)
- net N$4: now also U3a.15 (Q4)
- net N$8: no longer names the net of RN2.4 (R4.1)
- net N$8: now also U3b.12 (Q7)
- new net: U8.1 (IN), U8.13 (IN), U8.2 (IN)
- new net -5V_A: U8.10 (OUTS), U8.11 (OUT), U8.12 (OUT)
Other:
- moved on the sheet: J1

Commit message: Pack the schematics into a readable shape
Both sheets were strips: the main board ran 1765 mm wide across five bands,
the module 1509 across three, at aspect ratios of 6.4 and 10 to 1. Nothing
about that is followable.

Two changes. A cluster is now laid out as a compact block rather than a
single row, so twenty parts sharing a net form a scannable square instead of
a line. And the blocks are shelf-packed toward the proportions of a sheet of
paper rather than running rightward until a fixed width is hit.

The main board now reads as 663 by 706 mm across 14 bands, the module as 414
by 411 across 8. Roughly square rather than landscape, because shelf packing
wastes about a third of its area and the target is set to allow for that.

The sheet itself is now sized to its contents instead of a fixed 1600 by
1200, which was larger than A0 and part of why everything spread out.

Co-Authored-By: Claude Opus 5 <noreply@anthropic.com>
Connections:
- net +2V5: now also J1.1 (Pin_1), J1.10 (Pin_10), J1.11 (Pin_11), J1.12 (Pin_12), J1.13 (Pin_13), J1.14 (Pin_14), J1.15 (Pin_15), J1.16 (Pin_16), J1.17 (Pin_17), J1.18 (Pin_18), J1.19 (Pin_19), J1.2 (Pin_2), J1.20 (Pin_20), J1.21 (Pin_21), J1.22 (Pin_22), J1.23 (Pin_23), J1.24 (Pin_24), J1.25 (Pin_25), J1.26 (Pin_26), J1.27 (Pin_27), J1.28 (Pin_28), J1.29 (Pin_29), J1.3 (Pin_3), J1.30 (Pin_30), J1.31 (Pin_31), J1.32 (Pin_32), J1.33 (Pin_33), J1.34 (Pin_34), J1.35 (Pin_35), J1.36 (Pin_36), J1.37 (Pin_37), J1.38 (Pin_38), J1.39 (Pin_39), J1.4 (Pin_4), J1.40 (Pin_40), J1.41 (Pin_41), J1.42 (Pin_42), J1.43 (Pin_43), J1.44 (Pin_44), J1.45 (Pin_45), J1.46 (Pin_46), J1.47 (Pin_47), J1.48 (Pin_48), J1.49 (Pin_49), J1.5 (Pin_5), J1.50 (Pin_50), J1.51 (Pin_51), J1.52 (Pin_52), J1.53 (Pin_53), J1.54 (Pin_54), J1.55 (Pin_55), J1.56 (Pin_56), J1.57 (Pin_57), J1.58 (Pin_58), J1.59 (Pin_59), J1.6 (Pin_6), J1.60 (Pin_60), J1.61 (Pin_61), J1.62 (Pin_62), J1.63 (Pin_63), J1.64 (Pin_64), J1.65 (Pin_65), J1.66 (Pin_66), J1.67 (Pin_67), J1.68 (Pin_68), J1.69 (Pin_69), J1.7 (Pin_7), J1.70 (Pin_70), J1.72 (Pin_72), J1.74 (Pin_74), J1.76 (Pin_76), J1.78 (Pin_78), J1.8 (Pin_8), J1.80 (Pin_80), J1.9 (Pin_9), RN1.2 (R2.1), RN1.5 (R4.2), RN1.6 (R3.2), RN1.7 (R2.2), RN1.8 (R1.2), RN2.1 (R1.1), RN2.2 (R2.1), RN2.3 (R3.1), RN2.5 (R4.2), RN2.6 (R3.2), RN2.7 (R2.2), RN2.8 (R1.2), RN3.4 (R4.1), RN3.5 (R4.2), RN3.6 (R3.2), RN3.7 (R2.2), RN3.8 (R1.2), RN4.1 (R1.1), RN4.2 (R2.1), RN4.3 (R3.1), RN4.4 (R4.1), RN4.5 (R4.2), RN4.6 (R3.2), RN4.7 (R2.2), RN4.8 (R1.2), RN5.1 (R1.1), RN5.2 (R2.1), RN5.3 (R3.1), RN5.4 (R4.1), RN5.5 (R4.2), RN5.6 (R3.2), RN5.7 (R2.2), RN5.8 (R1.2), RN6.1 (R1.1), RN6.2 (R2.1), RN6.3 (R3.1), RN6.4 (R4.1), RN6.5 (R4.2), RN6.6 (R3.2), RN6.7 (R2.2), RN6.8 (R1.2), RN7.1 (R1.1), RN7.2 (R2.1), RN7.3 (R3.1), RN7.4 (R4.1), RN7.5 (R4.2), RN7.6 (R3.2), RN7.7 (R2.2), RN7.8 (R1.2), U1.1 (C), U1.4 (GND), U1.5 (Q), U2.10 (2B2), U2.11 (2B1), U2.12 (1B2), U2.13 (1B1), U2.14 (2~{OE}), U2.15 (1~{OE}), U2.2 (1DIR), U2.4 (1A1), U2.6 (2A1), U2.7 (2A2), U2.8 (GND), U2.9 (GND), U3a.1 (OE), U3a.10 (GND), U3a.13 (Q6), U3a.16 (Q3), U3a.17 (Q2), U3a.18 (Q1), U3a.2 (D0), U3a.3 (D1), U3a.4 (D2), U3a.5 (D3), U3a.6 (D4), U3a.7 (D5), U3a.8 (D6), U3b.1 (OE), U3b.10 (GND), U3b.16 (Q3), U3b.17 (Q2), U3b.18 (Q1), U3b.2 (D0), U3b.3 (D1), U3b.4 (D2), U3b.5 (D3), U3b.6 (D4), U3b.7 (D5), U3b.8 (D6), U4a.1 (OE), U4a.10 (GND), U4a.12 (Q7), U4a.13 (Q6), U4a.14 (Q5), U4a.15 (Q4), U4a.16 (Q3), U4a.17 (Q2), U4a.18 (Q1), U4a.2 (D0), U4a.3 (D1), U4a.4 (D2), U4a.5 (D3), U4a.6 (D4), U4a.7 (D5), U4a.8 (D6), U4b.1 (OE), U4b.10 (GND), U4b.12 (Q7), U4b.13 (Q6), U4b.14 (Q5), U4b.15 (Q4), U4b.16 (Q3), U4b.17 (Q2), U4b.18 (Q1), U4b.2 (D0), U4b.3 (D1), U4b.4 (D2), U4b.5 (D3), U4b.6 (D4), U4b.7 (D5), U4b.8 (D6), U5.11 (GND), U5.5 (ILIM), U5.8 (GND), U6.11 (GND), U6.5 (ILIM), U6.8 (GND), U8.9 (GND), U9.11 (GND), U9.5 (ILIM), U9.8 (GND), Y1.1 (EN), Y1.2 (GND), Y1.3 (OUT), Y2.1 (EN), Y2.2 (GND), Y2.3 (OUT); no longer U3a.20 (VCC), U3b.20 (VCC), U4a.20 (VCC), U4b.20 (VCC), U5.10 (OUT), U5.7 (SET), U5.9 (OUTS), U6.7 (SET), U9.7 (SET)
- removed net ELEM28: J1.1 (Pin_1), J1.10 (Pin_10), J1.11 (Pin_11), J1.12 (Pin_12), J1.13 (Pin_13), J1.14 (Pin_14), J1.15 (Pin_15), J1.16 (Pin_16), J1.17 (Pin_17), J1.18 (Pin_18), J1.19 (Pin_19), J1.2 (Pin_2), J1.20 (Pin_20), J1.21 (Pin_21), J1.22 (Pin_22), J1.23 (Pin_23), J1.24 (Pin_24), J1.25 (Pin_25), J1.26 (Pin_26), J1.27 (Pin_27), J1.28 (Pin_28), J1.29 (Pin_29), J1.3 (Pin_3), J1.30 (Pin_30), J1.31 (Pin_31), J1.32 (Pin_32), J1.33 (Pin_33), J1.34 (Pin_34), J1.35 (Pin_35), J1.36 (Pin_36), J1.37 (Pin_37), J1.38 (Pin_38), J1.39 (Pin_39), J1.4 (Pin_4), J1.40 (Pin_40), J1.41 (Pin_41), J1.42 (Pin_42), J1.43 (Pin_43), J1.44 (Pin_44), J1.45 (Pin_45), J1.46 (Pin_46), J1.47 (Pin_47), J1.48 (Pin_48), J1.49 (Pin_49), J1.5 (Pin_5), J1.50 (Pin_50), J1.51 (Pin_51), J1.52 (Pin_52), J1.53 (Pin_53), J1.54 (Pin_54), J1.55 (Pin_55), J1.56 (Pin_56), J1.57 (Pin_57), J1.58 (Pin_58), J1.59 (Pin_59), J1.6 (Pin_6), J1.60 (Pin_60), J1.61 (Pin_61), J1.62 (Pin_62), J1.63 (Pin_63), J1.64 (Pin_64), J1.65 (Pin_65), J1.66 (Pin_66), J1.67 (Pin_67), J1.68 (Pin_68), J1.69 (Pin_69), J1.7 (Pin_7), J1.70 (Pin_70), J1.72 (Pin_72), J1.74 (Pin_74), J1.76 (Pin_76), J1.78 (Pin_78), J1.8 (Pin_8), J1.80 (Pin_80), J1.9 (Pin_9), RN1.2 (R2.1), RN1.5 (R4.2), RN1.6 (R3.2), RN1.7 (R2.2), RN1.8 (R1.2), RN2.1 (R1.1), RN2.2 (R2.1), RN2.3 (R3.1), RN2.5 (R4.2), RN2.6 (R3.2), RN2.7 (R2.2), RN2.8 (R1.2), RN3.1 (R1.1), RN3.2 (R2.1), RN3.3 (R3.1), RN3.4 (R4.1), RN3.5 (R4.2), RN3.6 (R3.2), RN3.7 (R2.2), RN3.8 (R1.2), RN4.1 (R1.1), RN4.2 (R2.1), RN4.4 (R4.1), RN4.5 (R4.2), RN4.6 (R3.2), RN4.7 (R2.2), RN4.8 (R1.2), RN5.1 (R1.1), RN5.2 (R2.1), RN5.3 (R3.1), RN5.4 (R4.1), RN5.5 (R4.2), RN5.6 (R3.2), RN5.7 (R2.2), RN5.8 (R1.2), RN6.1 (R1.1), RN6.3 (R3.1), RN6.4 (R4.1), RN6.5 (R4.2), RN6.6 (R3.2), RN6.7 (R2.2), RN6.8 (R1.2), RN7.1 (R1.1), RN7.2 (R2.1), RN7.3 (R3.1), RN7.4 (R4.1), RN7.5 (R4.2), RN7.6 (R3.2), RN7.7 (R2.2), RN7.8 (R1.2), U1.1 (C), U1.4 (GND), U2.10 (2B2), U2.11 (2B1), U2.12 (1B2), U2.14 (2~{OE}), U2.15 (1~{OE}), U2.2 (1DIR), U2.4 (1A1), U2.6 (2A1), U2.7 (2A2), U2.8 (GND), U2.9 (GND), U3a.1 (OE), U3a.10 (GND), U3a.13 (Q6), U3a.16 (Q3), U3a.17 (Q2), U3a.18 (Q1), U3a.2 (D0), U3a.3 (D1), U3a.4 (D2), U3a.5 (D3), U3a.6 (D4), U3a.7 (D5), U3a.8 (D6), U3b.1 (OE), U3b.10 (GND), U3b.13 (Q6), U3b.14 (Q5), U3b.15 (Q4), U3b.16 (Q3), U3b.17 (Q2), U3b.18 (Q1), U3b.2 (D0), U3b.3 (D1), U3b.4 (D2), U3b.5 (D3), U3b.6 (D4), U3b.7 (D5), U3b.8 (D6), U4a.1 (OE), U4a.10 (GND), U4a.13 (Q6), U4a.14 (Q5), U4a.15 (Q4), U4a.16 (Q3), U4a.17 (Q2), U4a.18 (Q1), U4a.2 (D0), U4a.3 (D1), U4a.4 (D2), U4a.5 (D3), U4a.6 (D4), U4a.7 (D5), U4a.8 (D6), U4b.1 (OE), U4b.10 (GND), U4b.13 (Q6), U4b.14 (Q5), U4b.15 (Q4), U4b.16 (Q3), U4b.17 (Q2), U4b.18 (Q1), U4b.2 (D0), U4b.3 (D1), U4b.4 (D2), U4b.5 (D3), U4b.6 (D4), U4b.7 (D5), U4b.8 (D6), U5.11 (GND), U5.5 (ILIM), U5.8 (GND), U6.11 (GND), U6.5 (ILIM), U6.8 (GND), U8.9 (GND), U9.11 (GND), U9.5 (ILIM), U9.8 (GND), Y1.1 (EN), Y1.2 (GND), Y1.3 (OUT), Y2.1 (EN), Y2.2 (GND), Y2.3 (OUT)
- new net: RN3.1 (R1.1), U3b.13 (Q6)
- new net: RN3.2 (R2.1), U3b.14 (Q5)
- new net: RN3.3 (R3.1), U3b.15 (Q4)
- new net +3V3_REF: U3a.20 (VCC), U3b.20 (VCC), U4a.20 (VCC), U4b.20 (VCC), U5.10 (OUT), U5.9 (OUTS)
Other:
- moved on the sheet: C1, C10, C11, C12, C13, C14, C15, C16, C2, C3, C4, C5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
