File: hardware/lyrebird-main-reva/lyrebird-main.kicad_sch (KiCad schematic)
At the start: 133 parts, among them J1 Connfly DS1104-01, J2 Mezzanine 2x40, J3 JTAG 2x5 1.27mm, Q1 BSS138, U1 CCGM1A1-BGA324, U2 FT601Q, U3 LT3045, U4 LTM4622IV#PBF, U6 MX25R6435F 64Mb, Y1 ABM8G-30.000MHZ-18-D2Y-T

Commit message: Draw wires in the schematics instead of relying on net labels
Labels alone are hard to follow, so nets of two or three pins are now drawn
as wires and the parts sharing one are placed next to each other to keep the
wire short. That covers 119 of the main board's 125 nets and 68 of the
module's 82.

The split follows what a person does by hand rather than a rule of thumb.
Ground, the supply rails and the element bus stay as labels, because a wire
joining 245 ground pins is not a drawing anyone can read. Everything else is
a line you can trace.

Parts are clustered by the nets that join them, 94 clusters on the main board
and 19 on the module, so a wire is usually a short hop between neighbours
rather than a line across the sheet. Two-pin nets route as an L, three-pin
nets as a comb to a shared vertical. There is still no global routing, which
is the part that cannot be automated.

One bug had been silently eating most of the connectivity. KiCad symbols may
inherit from a base through `extends`, carrying its graphics and pins while
overriding properties. The reader took such a symbol at face value and saw no
pins at all, so 58 of 68 candidate nets on the module failed their pin lookup
and went unwired. Inheritance is now flattened before pins are read.

PDFs of both schematics are committed beside their boards.

Co-Authored-By: Claude Opus 5 <noreply@anthropic.com>
Parts:
- removed C11: 10nF, symbol Device:C
- removed C46: 100nF, symbol Device:C
- added J2: Mezzanine 2x40, symbol Connector_Generic:Conn_02x40_Odd_Even
- added U2: FT601Q, symbol Interface_USB:FT601Q
- C11: renamed from U2; value FT601Q -> 10nF; symbol Interface_USB:FT601Q -> Device:C
- C46: renamed from J2; value Mezzanine 2x40 -> 100nF; symbol Connector_Generic:Conn_02x40_Odd_Even -> Device:C
Connections:
- net CFG_DONE is gone; now on net +1V0: J3.7 (Pin_7)
- net CFG_FAILED_N is gone; now on net +1V0: J3.10 (Pin_10)
- net JTAG_TCK is gone; now on net +1V0: J3.4 (Pin_4)
- net JTAG_TDI is gone; now on net +1V0: J3.8 (Pin_8)
- net JTAG_TDO is gone; now on net +1V0: J3.6 (Pin_6)
- net JTAG_TMS is gone; now on net +1V0: J3.2 (Pin_2)
- net N$10 is gone; now on net +1V0: U4.A3 (TRACK/SS2)
- net N$2 is gone; now on net +1V0: J1.7 (SSTX+)
- net N$4 is gone; now on net +1V0: J1.6 (SSTX-)
- net N$6 is gone; now on an unnamed net: U4.E4 (FB1)
- net N$7 is gone; now on an unnamed net: U4.A4 (FB2)
- net N$8 is gone; now on net +1V0: U4.C4 (FREQ)
- net N$9 is gone; now on net +1V0: U4.E3 (TRACK/SS1)
- net PG_1 is gone; now on net +1V0: U4.D4 (PGOOD1)
- net PG_2 is gone; now on net +1V0: U4.B4 (PGOOD2)
- net SPI_CLK is gone; now on net +1V0: U6.6 (SCLK)
- net SPI_CS_N is gone; now on net +1V0: U6.1 (~{CS})
- net SPI_D0 is gone; now on net +1V0: U6.5 (SI/SIO0)
- net SPI_D1 is gone; now on net +1V0: U6.2 (SO/SIO1)
- net SPI_D2 is gone; now on net +1V0: U6.3 (~{WP}/SIO2)
- net SPI_D3 is gone; now on net +1V0: U6.7 (~{RESET}/SIO3)
- net USB_VBUS is gone; now on net +1V0: J1.1 (VBUS)
- net +1V0: now also J1.10 (SSRX+), J1.2 (D-), J1.3 (D+), J1.5 (GND), J1.8 (DRAIN), J1.9 (SSRX-), J1.SH (SHIELD), J3.1 (Pin_1), J3.3 (Pin_3), J3.5 (Pin_5), J3.9 (Pin_9), Q1.1 (G), Q1.2 (S), U1.V13 (SER_TX_N), U3.1 (IN), U3.11 (GND), U3.2 (IN), U3.3 (EN/UV), U3.5 (ILIM), U3.6 (PGFB), U3.8 (GND), U4.A2 (VIN2), U4.B3 (VIN2), U4.B5 (GND), U4.C1 (GND), U4.C2 (GND), U4.C5 (SYNC/MODE), U4.D1 (VOUT1), U4.D2 (RUN1), U4.D3 (VIN1), U4.D5 (GND), U4.E1 (VOUT1), U4.E2 (VIN1), U6.4 (GND), U6.8 (VCC), Y1.2 (G), Y1.4 (G), J2.1 (Pin_1), J2.10 (Pin_10), J2.11 (Pin_11), J2.12 (Pin_12), J2.13 (Pin_13), J2.14 (Pin_14), J2.15 (Pin_15), J2.16 (Pin_16), J2.17 (Pin_17), J2.18 (Pin_18), J2.19 (Pin_19), J2.2 (Pin_2), J2.20 (Pin_20), J2.21 (Pin_21), J2.22 (Pin_22), J2.23 (Pin_23), J2.24 (Pin_24), J2.25 (Pin_25), J2.26 (Pin_26), J2.27 (Pin_27), J2.28 (Pin_28), J2.29 (Pin_29), J2.3 (Pin_3), J2.30 (Pin_30), J2.31 (Pin_31), J2.32 (Pin_32), J2.33 (Pin_33), J2.34 (Pin_34), J2.35 (Pin_35), J2.36 (Pin_36), J2.37 (Pin_37), J2.38 (Pin_38), J2.39 (Pin_39), J2.4 (Pin_4), J2.40 (Pin_40), J2.41 (Pin_41), J2.42 (Pin_42), J2.43 (Pin_43), J2.44 (Pin_44), J2.45 (Pin_45), J2.46 (Pin_46), J2.47 (Pin_47), J2.48 (Pin_48), J2.49 (Pin_49), J2.5 (Pin_5), J2.50 (Pin_50), J2.51 (Pin_51), J2.52 (Pin_52), J2.53 (Pin_53), J2.54 (Pin_54), J2.55 (Pin_55), J2.56 (Pin_56), J2.57 (Pin_57), J2.58 (Pin_58), J2.59 (Pin_59), J2.6 (Pin_6), J2.60 (Pin_60), J2.61 (Pin_61), J2.62 (Pin_62), J2.63 (Pin_63), J2.64 (Pin_64), J2.65 (Pin_65), J2.66 (Pin_66), J2.67 (Pin_67), J2.68 (Pin_68), J2.69 (Pin_69), J2.7 (Pin_7), J2.70 (Pin_70), J2.71 (Pin_71), J2.72 (Pin_72), J2.73 (Pin_73), J2.74 (Pin_74), J2.75 (Pin_75), J2.76 (Pin_76), J2.77 (Pin_77), J2.78 (Pin_78), J2.79 (Pin_79), J2.8 (Pin_8), J2.80 (Pin_80), J2.9 (Pin_9), U2.1 (GND), U2.10 (~{SIWU}), U2.11 (~{WR}), U2.12 (~{RD}), U2.13 (~{OE}), U2.14 (VCCIO), U2.15 (~{RESET}), U2.16 (~{WAKEUP}), U2.17 (GPIO0), U2.18 (GPIO1), U2.21 (XI), U2.22 (XO), U2.23 (DP), U2.25 (DM), U2.26 (GND), U2.27 (RREF), U2.29 (GND), U2.31 (TODN), U2.32 (TODP), U2.34 (RIDN), U2.35 (RIDP), U2.36 (GND), U2.37 (VBUS), U2.4 (BE_0), U2.40 (DATA_0), U2.41 (DATA_1), U2.42 (DATA_2), U2.43 (DATA_3), U2.44 (DATA_4), U2.45 (DATA_5), U2.46 (DATA_6), U2.47 (DATA_7), U2.49 (VCCIO), U2.5 (BE_1), U2.50 (DATA_8), U2.51 (DATA_9), U2.52 (DATA_10), U2.53 (DATA_11), U2.54 (DATA_12), U2.55 (DATA_13), U2.56 (DATA_14), U2.57 (DATA_15), U2.58 (CLK), U2.59 (VCCIO), U2.6 (BE_2), U2.60 (DATA_16), U2.61 (DATA_17), U2.62 (DATA_18), U2.63 (DATA_19), U2.64 (DATA_20), U2.65 (DATA_21), U2.66 (DATA_22), U2.67 (DATA_23), U2.68 (VCCIO), U2.69 (DATA_24), U2.7 (BE_3), U2.70 (DATA_25), U2.71 (DATA_26), U2.72 (DATA_27), U2.73 (DATA_28), U2.74 (DATA_29), U2.75 (DATA_30), U2.76 (DATA_31), U2.77 (GND), U2.8 (~{TXE}), U2.9 (~{RXF})
- net +1V0_FT: now also U2.2 (AVDD), U2.3 (VD10), U2.30 (VD10), U2.33 (VD10), U2.39 (DV10), U2.48 (VD10); no longer C11.2 (AVDD), C11.3 (VD10), C11.30 (VD10), C11.33 (VD10), C11.39 (DV10), C11.48 (VD10)
- net +3V3: now also U2.20 (VCC33), U2.24 (VCC33), U2.28 (VDDA), U2.38 (VCC33); no longer C11.20 (VCC33), C11.24 (VCC33), C11.28 (VDDA), C11.38 (VCC33)
- removed net +2V5: C11.14 (VCCIO), C11.49 (VCCIO), C11.59 (VCCIO), C11.68 (VCCIO), J3.1 (Pin_1), U1.V13 (SER_TX_N), U4.D1 (VOUT1), U4.E1 (VOUT1), U6.8 (VCC)
- removed net +5V: C11.37 (VBUS), C46.71 (Pin_71), C46.73 (Pin_73), C46.75 (Pin_75), C46.77 (Pin_77), C46.79 (Pin_79), U3.1 (IN), U3.2 (IN), U3.3 (EN/UV), U3.6 (PGFB), U4.A2 (VIN2), U4.B3 (VIN2), U4.D2 (RUN1), U4.D3 (VIN1), U4.E2 (VIN1)
- net CORE_RUN: no longer names the net of U4.B2 (RUN2)
- net CORE_RUN: now also Q1.3 (D)
- net ELEM0: no longer names the net of C46.1
- net ELEM0: no longer C11.41 (DATA_1)
- removed net ELEM1: C11.46 (DATA_6), C46.3 (Pin_3), C46.61 (Pin_61)
- removed net ELEM10: C11.40 (DATA_0), C46.21 (Pin_21)
- removed net ELEM11: C11.52 (DATA_10), C46.23 (Pin_23), C46.57 (Pin_57)
- removed net ELEM12: C11.53 (DATA_11), C46.25 (Pin_25), C46.49 (Pin_49)
- removed net ELEM13: C11.55 (DATA_13), C11.8 (~{TXE}), C46.27 (Pin_27), C46.41 (Pin_41)
- removed net ELEM14: C11.44 (DATA_4), C46.29 (Pin_29)
- removed net ELEM15: C11.56 (DATA_14), C46.31 (Pin_31), C46.59 (Pin_59)
- removed net ELEM16: C11.57 (DATA_15), C46.33 (Pin_33), C46.51 (Pin_51)
- removed net ELEM17: C11.61 (DATA_17), C11.9 (~{RXF}), C46.35 (Pin_35), C46.43 (Pin_43)
- removed net ELEM18: C11.11 (~{WR}), C11.43 (DATA_3), C46.37 (Pin_37), C46.9 (Pin_9)
- removed net ELEM19: C11.12 (~{RD}), C11.50 (DATA_8), C46.19 (Pin_19), C46.39 (Pin_39)
- removed net ELEM2: C11.42 (DATA_2), C46.5 (Pin_5), C46.53 (Pin_53)
- removed net ELEM22: C11.10 (~{SIWU}), C11.54 (DATA_12), C46.45 (Pin_45), C46.7 (Pin_7)
- removed net ELEM23: C11.13 (~{OE}), C11.60 (DATA_16), C46.17 (Pin_17), C46.47 (Pin_47)
- removed net ELEM27: C11.47 (DATA_7), C46.15 (Pin_15), C46.55 (Pin_55)
- removed net ELEM31: C11.51 (DATA_9), C46.13 (Pin_13), C46.63 (Pin_63)
- removed net ELEM5: C11.45 (DATA_5), C46.11 (Pin_11)
- removed net FT_BE0: C11.4 (BE_0)
- removed net FT_BE1: C11.5 (BE_1), C46.70 (Pin_70)
- removed net FT_BE2: C11.6 (BE_2)
- removed net FT_BE3: C11.58 (CLK), C11.7 (BE_3), C46.66 (Pin_66)
- removed net FT_DATA18: C11.62 (DATA_18)
- removed net FT_DATA19: C11.63 (DATA_19)
- removed net FT_DATA20: C11.64 (DATA_20)
- removed net FT_DATA21: C11.65 (DATA_21), C46.69 (Pin_69)
- removed net FT_DATA22: C11.66 (DATA_22)
- removed net FT_DATA23: C11.67 (DATA_23)
- removed net FT_DATA24: C11.69 (DATA_24)
- removed net FT_DATA25: C11.70 (DATA_25), C46.65 (Pin_65), C46.68 (Pin_68)
- removed net FT_DATA26: C11.71 (DATA_26)
- removed net FT_DATA27: C11.72 (DATA_27)
- removed net FT_DATA28: C11.73 (DATA_28)
- removed net FT_DATA29: C11.74 (DATA_29)
- removed net FT_DATA30: C11.75 (DATA_30), C46.67 (Pin_67)
- removed net FT_DATA31: C11.76 (DATA_31)
- removed net FT_GPIO0: C11.17 (GPIO0)
- removed net FT_GPIO1: C11.18 (GPIO1)
- removed net FT_RESET_N: C11.15 (~{RESET})
- removed net FT_RREF: C11.27 (RREF)
- removed net FT_WAKEUP_N: C11.16 (~{WAKEUP})
- removed net FT_XI: C11.21 (XI)
- removed net FT_XO: C11.22 (XO)
- removed net GND: C11.1 (GND), C11.26 (GND), C11.29 (GND), C11.36 (GND), C11.77 (GND), C46.10 (Pin_10), C46.12 (Pin_12), C46.14 (Pin_14), C46.16 (Pin_16), C46.18 (Pin_18), C46.2 (Pin_2), C46.20 (Pin_20), C46.22 (Pin_22), C46.24 (Pin_24), C46.26 (Pin_26), C46.28 (Pin_28), C46.30 (Pin_30), C46.32 (Pin_32), C46.34 (Pin_34), C46.36 (Pin_36), C46.38 (Pin_38), C46.4 (Pin_4), C46.40 (Pin_40), C46.42 (Pin_42), C46.44 (Pin_44), C46.46 (Pin_46), C46.48 (Pin_48), C46.50 (Pin_50), C46.52 (Pin_52), C46.54 (Pin_54), C46.56 (Pin_56), C46.58 (Pin_58), C46.6 (Pin_6), C46.60 (Pin_60), C46.62 (Pin_62), C46.64 (Pin_64), C46.72 (Pin_72), C46.74 (Pin_74), C46.76 (Pin_76), C46.78 (Pin_78), C46.8 (Pin_8), C46.80 (Pin_80), J1.5 (GND), J1.8 (DRAIN), J1.SH (SHIELD), J3.3 (Pin_3), J3.5 (Pin_5), J3.9 (Pin_9), U3.11 (GND), U3.5 (ILIM), U3.8 (GND), U4.B5 (GND), U4.C1 (GND), U4.C2 (GND), U4.C5 (SYNC/MODE), U4.D5 (GND), U6.4 (GND), Y1.2 (G), Y1.4 (G)
- removed net N$1: C11.32 (TODP)
- removed net N$3: C11.31 (TODN)
- net N$5: no longer names the net of U3.7 (SET)
- removed net USB_DM: C11.25 (DM), J1.2 (D-)
- removed net USB_DP: C11.23 (DP), J1.3 (D+)
- removed net USB_SSRX_N: C11.34 (RIDN), J1.9 (SSRX-)
- removed net USB_SSRX_P: C11.35 (RIDP), J1.10 (SSRX+)

Commit message: Pack the schematics into a readable shape
Both sheets were strips: the main board ran 1765 mm wide across five bands,
the module 1509 across three, at aspect ratios of 6.4 and 10 to 1. Nothing
about that is followable.

Two changes. A cluster is now laid out as a compact block rather than a
single row, so twenty parts sharing a net form a scannable square instead of
a line. And the blocks are shelf-packed toward the proportions of a sheet of
paper rather than running rightward until a fixed width is hit.

The main board now reads as 663 by 706 mm across 14 bands, the module as 414
by 411 across 8. Roughly square rather than landscape, because shelf packing
wastes about a third of its area and the target is set to allow for that.

The sheet itself is now sized to its contents instead of a fixed 1600 by
1200, which was larger than A0 and part of why everything spread out.

Co-Authored-By: Claude Opus 5 <noreply@anthropic.com>
Connections:
- net +3V3 is gone; now on net +1V0: U2.20 (VCC33), U2.24 (VCC33), U2.28 (VDDA), U2.38 (VCC33), U3.10 (OUT), U3.9 (OUTS)
- net +1V0: now also U4.E4 (FB1); no longer J1.1 (VBUS), J1.6 (SSTX-)
- net at Q1.3 (D), U4.A4 (FB2), U4.B2 (RUN2): no longer U4.E4 (FB1)
Other:
- moved on the sheet: C1, C10, C100, C11, C12, C13, C14, C15, C16, C17, C18, C19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
