File: hardware/lyrebird-main-reva/sheets/01-U1-CCGM1A1-BGA324.kicad_sch (KiCad schematic)
At the start: 87 parts, among them U1 CCGM1A1-BGA324

Commit message: Regenerate the schematics, which were eleven days behind the netlists
The sheets and both PDFs dated 13 September against netlists from
today. They showed a board with USB bus power, a charge pump on the
analog module, no JTAG series protection, no oscillator pull-downs and
none of the footprint corrections -- a board that has not existed for
some time. Anyone opening them to review the design would have been
reviewing the wrong one, which is worse than having no schematic.

Regenerated from the current netlists: the main board goes from 8
sheets to 11, picking up the wall-wart input and the inverter, and the
module from 6 to 9 while losing the charge pump entirely. Both PDFs
rebuilt through kicad-cli, one page per sheet.

Nothing regenerated them because nothing was watching. The netlist
generators are run constantly and the views derived from them are not,
so they drift silently and there is no check that notices.

Co-Authored-By: Claude Opus 5 <noreply@anthropic.com>
Parts:
- added R26, R28, R30: 10k, symbol Device:R
- C101: renamed from C15; value 22uF -> 100nF
- C102: renamed from C16; value 22uF -> 100nF
- C24, C25: value 100nF -> 22uF
- renumbered C20 to C106, C21 to C107, C22 to C108, C23 to C109, C19 to C28, C26 to C29, C27 to C30, C28 to C31, C29 to C32, C30 to C33, C31 to C34, C32 to C35, C33 to C36, C34 to C37, C35 to C38, C36 to C39, C37 to C40, C38 to C41, C39 to C42, C40 to C43, C41 to C44, C42 to C45, C43 to C46, C44 to C47, C45 to C48, C46 to C49, C47 to C50, C48 to C51, C49 to C52, C50 to C53, C51 to C54, C52 to C55, C53 to C56, C54 to C57, C55 to C58, C56 to C59, C57 to C60, C58 to C61, C59 to C62, C60 to C63, C61 to C64, C62 to C65, C63 to C66, C64 to C67, C65 to C68, C66 to C69, C67 to C70, C68 to C71, C69 to C72, C70 to C73, C71 to C74, C72 to C75, C73 to C76, C74 to C77, C75 to C78, C76 to C79, C77 to C80, C78 to C81, C79 to C82, C80 to C83, C81 to C84, C82 to C85, C83 to C86, C84 to C87, C85 to C88, C86 to C89, C87 to C90, C88 to C91, C89 to C92, C90 to C93, C91 to C94, C92 to C95, C93 to C96, R13 to R17, R16 to R22, R17 to R23, R18 to R24, R19 to R25
Connections:
- net GND: now also U1.V11 (SER_RX_N)
Other:
- moved on the sheet: C109, C24, C25, C29, C30, C31, C32, C33, C34, C35, C36, C37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
