File: hardware/lyrebird-main-reva/sheets/03-U4-LTM4622IVPBF.kicad_sch (KiCad schematic)
At the start: 9 parts, among them U4 LTM4622IV#PBF

Commit message: Regenerate the schematics, which were eleven days behind the netlists
The sheets and both PDFs dated 13 September against netlists from
today. They showed a board with USB bus power, a charge pump on the
analog module, no JTAG series protection, no oscillator pull-downs and
none of the footprint corrections -- a board that has not existed for
some time. Anyone opening them to review the design would have been
reviewing the wrong one, which is worse than having no schematic.

Regenerated from the current netlists: the main board goes from 8
sheets to 11, picking up the wall-wart input and the inverter, and the
module from 6 to 9 while losing the charge pump entirely. Both PDFs
rebuilt through kicad-cli, one page per sheet.

Nothing regenerated them because nothing was watching. The netlist
generators are run constantly and the views derived from them are not,
so they drift silently and there is no check that notices.

Co-Authored-By: Claude Opus 5 <noreply@anthropic.com>
Parts:
- added C18: 10uF, symbol Device:C
- added C22, C23: 4.7uF, symbol Device:C
- added R1: 100k, symbol Device:R
- C12: renamed from R8; value 100k -> 47uF; symbol Device:R -> Device:C
- R10: renamed from R2; value 19.1k 1% -> 649k 1%
- R11: renamed from R3; value 90.9k 1% -> 100k
- R12: renamed from R4; value 649k 1% -> 100k
- R8: renamed from R5; value 100k -> 19.1k 1%
- R9: renamed from R6; value 100k -> 90.9k 1%
- renumbered C11 to C20, C12 to C21
Connections:
- net +2V5: no longer U4.A4 (FB2), U4.B2 (RUN2)
- net +5V: now also U4.A4 (FB2), U4.B2 (RUN2)
