File: hardware/lyrebird-main-reva/sheets/09-U3-LT3045.kicad_sch (KiCad schematic)
At the start: 3 parts, among them U3 LT3045

Commit message: Regenerate the schematics, which were eleven days behind the netlists
The sheets and both PDFs dated 13 September against netlists from
today. They showed a board with USB bus power, a charge pump on the
analog module, no JTAG series protection, no oscillator pull-downs and
none of the footprint corrections -- a board that has not existed for
some time. Anyone opening them to review the design would have been
reviewing the wrong one, which is worse than having no schematic.

Regenerated from the current netlists: the main board goes from 8
sheets to 11, picking up the wall-wart input and the inverter, and the
module from 6 to 9 while losing the charge pump entirely. Both PDFs
rebuilt through kicad-cli, one page per sheet.

Nothing regenerated them because nothing was watching. The netlist
generators are run constantly and the views derived from them are not,
so they drift silently and there is no check that notices.

Co-Authored-By: Claude Opus 5 <noreply@anthropic.com>
Parts:
- C17: renamed from C8; value 4.7uF -> 100nF
- renumbered R1 to R7
Changed lines of the file:
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@@
 	(symbol (lib_id "Device:C") (at 45.72 35.56 0) (unit 1)
 		(exclude_from_sim no) (in_bom yes) (on_board yes) (dnp no)
-		(property "Reference" "C8" (at 45.72 25.250000000000004 0)
+		(property "Reference" "C17" (at 45.72 25.250000000000004 0)
 			(effects (font (size 1.27 1.27))))
-		(property "Value" "4.7uF" (at 45.72 45.870000000000005 0)
+		(property "Value" "100nF" (at 45.72 45.870000000000005 0)
 			(effects (font (size 1.27 1.27))))
-		(instances (project "" (path "/" (reference "C8") (unit 1))))
+		(instances (project "" (path "/" (reference "C17") (unit 1))))
 	)
 	(symbol (lib_id "Device:R") (at 86.36 35.56 0) (unit 1)
 		(exclude_from_sim no) (in_bom yes) (on_board yes) (dnp no)
-		(property "Reference" "R1" (at 86.36 25.250000000000004 0)
+		(property "Reference" "R7" (at 86.36 25.250000000000004 0)
 			(effects (font (size 1.27 1.27))))
 		(property "Value" "33.2k 0.1%" (at 86.36 45.870000000000005 0)
 			(effects (font (size 1.27 1.27))))
-		(instances (project "" (path "/" (reference "R1") (unit 1))))
+		(instances (project "" (path "/" (reference "R7") (unit 1))))
 	)
 	(symbol (lib_id "Regulator_Linear:LT3045xDD") (at 45.72 73.66 0) (unit 1)
