File: hardware/lyrebird-main-reva/sheets/08-Other.kicad_sch (KiCad schematic)
At the start: 3 parts, among them J4 12 V 2.1 x 5.5 mm, centre pos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

Commit message: Check whether the documents still describe the boards, and rebuild the BOMs
Three times now the same failure has been found by accident: schematics
eleven days behind the netlists, a simulation asserting failures
against circuits already fixed, and power.md still listing AVDD on
+3V3 -- a destroy-the-part bug the netlist corrected long ago and the
document went on documenting. The netlist generators run constantly,
everything derived from them runs occasionally, and nothing compared
the two.

hardware/check_freshness.py compares them. Timestamps first, which are
cheap and weak -- a derived file older than its source is definitely
stale, a newer one only means somebody ran something. Then BOM
coverage against the netlist, which catches parts added or revalued
without the BOM following. Then a scan for superseded strings, which is
the only one of the three that can catch prose.

It found the BOMs were not merely stale but describing different
boards. The main board's listed three integrated circuits for a board
with seven, and no diodes, fuse, inductors or connectors at all. The
module's still named U3a, U3b, U4a and U4b, references that stopped
existing when the register symbol changed.

So the BOMs are generated now, by hardware/make_bom.py, from the
netlist. References, values and footprints are derived; manufacturer,
part number and the reason for the choice are annotated by reference,
and a part with no annotation is reported rather than quietly omitted.
That reporting immediately found two, both LT3045s whose values
differed from their siblings.

The Status column is the point of the file. This project has been
confidently wrong about a fuse that did not exist at its own rail
voltage and a footprint with the wrong lead count, so VERIFIED means a
datasheet was fetched and read, and UNVERIFIED means it was not.

One of my own rules was a false positive and is fixed: DFN-12 flagged
the LT3094, for which it is correct. It now requires LT3045 on the same
line.

Schem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
Parts:
- F1: value PTC >=24Vdc, 0.5 A hold, Imax >=40 A — PART UNCHOSEN -> 1812L050/30 PPTC 0.5A hold 30V 100A
Changed lines of the file:
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@@
 		(property "Reference" "F1" (at 35.56 25.250000000000004 0)
 			(effects (font (size 1.27 1.27))))
-		(property "Value" "PTC >=24Vdc, 0.5 A hold, Imax >=40 A — PART UNCHOSEN" (at 35.56 45.870000000000005 0)
+		(property "Value" "1812L050/30 PPTC 0.5A hold 30V 100A" (at 35.56 45.870000000000005 0)
 			(effects (font (size 1.27 1.27))))
 		(instances (project "" (path "/" (reference "F1") (unit 1))))
