File: hardware/lyrebird-main-reva/sheets/05-6-V-for-the-modules-analog-stage-0015.kicad_sch (KiCad schematic)
At the start: 7 parts, among them U7 LMR33630 12V->-6V inverting

Commit message: Write the decision record everything was already citing, and strike a claim
Twelve files referred to "decision 5" and no such record existed. The
phrase originated in a code comment and propagated into the decision
index itself, where a bare "5" reads as 0005. It is 0015 now -- the
negative rail crossing the mezzanine -- and every reference points at it.
Writing it closed five separate flags at once, because it was the missing
live home for all of them.

0014 claimed a "second 1.1 dB nobody was looking for" from a
noise-optimal element resistor at 2585 ohm. I wrote that and it is wrong
twice over, which a validation pass established and I confirmed by
recomputing:

  * 2585 ohm is not an optimum. run_analog.py solves
    1k * 10^((S_elem(1k) - floor)/10) for where the element resistors'
    own thermal noise equals the digital floor. No derivative, no argmax,
    and snr_elem_db is monotone in R -- 137.60 dB at 1k falling to
    130.88 at 4.7k. Lower is always quieter and always costs current.
    There is nothing to be at an optimum of.
  * The figure is 0.67 dB, not 1.1. The 1.1 is the element resistors
    measured alone; through the stage it is 126.50 against 125.83.

Struck in place rather than quietly restated, in 0014 and in the module's
power page. What survives is that the one-unit-load rule really is
retired, so the value can be revisited for about 0.67 dB.

Three other corrections from the same pass. 0014 specified a 15 V TVS
where the board fits the 18 V part it was changed to. 0013 carried a
git-lfs row reading "missing" two rows below one reading "installed",
which its own correction claimed to have fixed. And parts-notes.md still
described U14 as sitting on the pump's 5.69 V output programmed to
4.99 V -- the exact paragraph that documented the fault -- now corrected
with the fault recorded as a quotation beside it.

The freshness checker's worst hole is closed, and it was mine:
SUPERSEDED_OK exempted docs/decisions/ wholesale, so the only content
che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
Other:
- title: 6 V for the module's analog stage (decision 5, option B) -> 6 V for the module's analog stage (0015)
Changed lines of the file:
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@@
 	(generator "lyrebird")
 	(paper "User" 164 148)
-	(title_block (title "6 V for the module's analog stage (decision 5, option B)"))
+	(title_block (title "6 V for the module's analog stage (0015)"))
 	(symbol (lib_id "Device:C") (at 45.72 35.56 0) (unit 1)
 		(exclude_from_sim no) (in_bom yes) (on_board yes) (dnp no)
