File: hardware/lyrebird-main-reva/sheets/06-6-V-for-the-modules-analog-stage-0015.kicad_sch (KiCad schematic)
At the start: 7 parts, among them U7 LMR33630 12V->-6V inverting

Commit message: Act on the schematic validation: three faults and the core-rail guard
**The SuperSpeed pairs were wired backwards, and are now not wired.**
USB_SSRX_P/N were the only multi-node nets on the board with an INPUT at
every pin -- the receptacle's SSRX pins are inputs and so are the
bridge's RIDP/RIDN, so nothing drove them, and the transmit pair was
mirrored the same way. The comment asserted a crossover inside the cable
as fact and reasoned from it; USB 3.0 cables have no crossover.
SuperSpeed would never have trained and the link would have fallen back
to 480 Mb/s silently -- which is the speed 0014 chose on purpose, since
no galvanic isolator exists above USB 2.0. So the pairs are removed
rather than corrected, which also retires the hardest constraint in this
board's layout. How to wire them correctly if they ever come back is
recorded where they were.

**The inverting converter had no input capacitor across its own
terminals.** Nothing spanned +12V and -6V_A, and U7's GND pin *is*
-6V_A, so the loop its switching current actually takes was unbypassed
-- the input caps near U5 are referenced to system ground and are not in
that loop at all. This is the third fault found in U7 and all three are
the same mistake: reasoning about it as though its ground were the
board's.

**The translator's output enables are tied low against an explicit
datasheet instruction**, and the fix is sequencing rather than a pull-up.
SCES576I says OE must be pulled up to VCCA and not enabled until both
supplies are stable; a pull-up is not available here because nothing on
the module could pull it down -- no spare mezzanine pin, and MUTE_N has
the wrong polarity. Instead VCC(A) is made the last rail to arrive:
10 uF on U9's SET gives 573 ms against 359 ms for VCC(B), so the enable
cannot precede the supply it switches to. It costs nothing, because that
rail feeds the translator's reference supply and nothing else.

**The core rail now has a guard, and it needed two attempts.** The
existing as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
Parts:
- renumbered C13 to C11, C14 to C12
Changed lines of the file:
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@@
 	(symbol (lib_id "Device:C") (at 45.72 35.56 0) (unit 1)
 		(exclude_from_sim no) (in_bom yes) (on_board yes) (dnp no)
-		(property "Reference" "C13" (at 45.72 25.250000000000004 0)
+		(property "Reference" "C11" (at 45.72 25.250000000000004 0)
 			(effects (font (size 1.27 1.27))))
 		(property "Value" "1uF" (at 45.72 45.870000000000005 0)
 			(effects (font (size 1.27 1.27))))
-		(instances (project "" (path "/" (reference "C13") (unit 1))))
+		(instances (project "" (path "/" (reference "C11") (unit 1))))
 	)
 	(symbol (lib_id "Device:C") (at 86.36 35.56 0) (unit 1)
 		(exclude_from_sim no) (in_bom yes) (on_board yes) (dnp no)
-		(property "Reference" "C14" (at 86.36 25.250000000000004 0)
+		(property "Reference" "C12" (at 86.36 25.250000000000004 0)
 			(effects (font (size 1.27 1.27))))
 		(property "Value" "100nF" (at 86.36 45.870000000000005 0)
 			(effects (font (size 1.27 1.27))))
-		(instances (project "" (path "/" (reference "C14") (unit 1))))
+		(instances (project "" (path "/" (reference "C12") (unit 1))))
 	)
 	(symbol (lib_id "Device:L") (at 114.3 35.56 0) (unit 1)
@@
 		(instances (project "" (path "/" (reference "U7") (unit 1))))
 	)
+	(wire (pts (xy 45.72 33.02) (xy 45.72 111.76))
+		(stroke (width 0) (type default)))
+	(wire (pts (xy 45.72 111.76) (xy 35.56 111.76))
+		(stroke (width 0) (type default)))
+	(wire (pts (xy 86.36 40.64) (xy 86.36 101.6))
+		(stroke (width 0) (type default)))
+	(wire (pts (xy 86.36 101.6) (xy 55.88 101.6))
+		(stroke (width 0) (type default)))
 	(wire (pts (xy 86.36 66.04) (xy 86.36 109.22))
 		(stroke (width 0) (type default)))
@@
 	(junction (at 86.36 109.22) (diameter 0)
 		(color 0 0 0 0))
-	(wire (pts (xy 45.72 33.02) (xy 45.72 111.76))
-		(stroke (width 0) (type default)))
-	(wire (pts (xy 45.72 111.76) (xy 35.56 111.76))
-		(stroke (width 0) (type default)))
-	(wire (pts (xy 86.36 40.64) (xy 86.36 101.6))
-		(stroke (width 0) (type default)))
-	(wire (pts (xy 86.36 101.6) (xy 55.88 101.6))
-		(stroke (width 0) (type default)))
 	(wire (pts (xy 45.72 66.04) (xy 45.72 111.76))
 		(stroke (width 0) (type default)))
