File: hardware/lyrebird-dac-reva/sheets/04-The-bipolar-rail-decision-5-option-B-supersedes-.kicad_sch (KiCad schematic)
At the start: 11 parts, among them U14 LT3045 op amp positive rail, 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, U8 LT3094 op amp negative rail

Commit message: Fix a rail programmed above what its input can deliver
The documentation validator found an electrical fault, which is not
where one expects to find one. U14, the module's positive analog
regulator, had its SET resistor at 49.9k -- programming 4.99 V -- and I
had moved its input from the charge pump's 5.69 V to the header's 5.02 V
without touching it. Thirty millivolts of headroom against a part whose
published dropout is 260 mV at 500 mA. The rail would not have reached
its programmed voltage.

45.3k now, for 4.53 V and 490 mV of headroom. The stage needs far less
than either: it swings +/-2.83 V peak and the OPA1612 reaches within
600 mV of its rails, so 3.43 V would do. The rails are deliberately
asymmetric at +4.53 and -4.99, which costs nothing -- both clear the
swing, and matching the negative one down would add 30 mW in the LT3094
for no benefit.

What let it through is the more useful finding. verify_power.py's
dropout check tested the main board's LT3045, which has 1.7 V of
headroom and therefore could not fail, and none of the module's five
regulators. A check over one instance of a part is not a check over the
design. It now reads every LT3045 and LT3094 out of both netlists, takes
the programmed voltage from the SET resistor and the input from the rail
the IN pin sits on, and checks all six. Tamper-tested by restoring the
49.9k: U14 fails, 17 of 18.

Reading it from the netlist rather than restating the voltages here is
deliberate, and the fault is the argument -- a constant in this file
would have been left behind exactly as the resistor was.

One incidental lesson. My first version of that reader looked for
pinfunction fields, which this netlist does not contain at all, so it
returned no regulators and the suite passed 12 of 12 with the check
silently finding nothing to check. A check that locates no subjects
reports success.

Co-Authored-By: Claude Opus 5 <noreply@anthropic.com>
Parts:
- R10: value 49.9k 0.1% -> 45.3k 0.1%
- U14: value LT3045 op amp positive rail, +4.94 V from mezzanine 5 V -> LT3045 op amp positive rail, +4.53 V from mezzanine 5 V
Changed lines of the file:
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@@
 		(property "Reference" "R10" (at 86.36 114.15 0)
 			(effects (font (size 1.27 1.27))))
-		(property "Value" "49.9k 0.1%" (at 86.36 134.77 0)
+		(property "Value" "45.3k 0.1%" (at 86.36 134.77 0)
 			(effects (font (size 1.27 1.27))))
 		(instances (project "" (path "/" (reference "R10") (unit 1))))
@@
 		(property "Reference" "U14" (at 45.72 149.71 0)
 			(effects (font (size 1.27 1.27))))
-		(property "Value" "LT3045 op amp positive rail, +4.94 V from mezzanine 5 V" (at 45.72 175.41 0)
+		(property "Value" "LT3045 op amp positive rail, +4.53 V from mezzanine 5 V" (at 45.72 175.41 0)
 			(effects (font (size 1.27 1.27))))
 		(instances (project "" (path "/" (reference "U14") (unit 1))))
