File: hardware/lyrebird-dac-reva/sheets/04-The-bipolar-rail-0015-superseding-0009s.kicad_sch (KiCad schematic)
At the start: 11 parts, among them U14 LT3045 op amp positive rail, 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, U8 LT3094 op amp negative rail

Commit message: Write the decision record everything was already citing, and strike a claim
Twelve files referred to "decision 5" and no such record existed. The
phrase originated in a code comment and propagated into the decision
index itself, where a bare "5" reads as 0005. It is 0015 now -- the
negative rail crossing the mezzanine -- and every reference points at it.
Writing it closed five separate flags at once, because it was the missing
live home for all of them.

0014 claimed a "second 1.1 dB nobody was looking for" from a
noise-optimal element resistor at 2585 ohm. I wrote that and it is wrong
twice over, which a validation pass established and I confirmed by
recomputing:

  * 2585 ohm is not an optimum. run_analog.py solves
    1k * 10^((S_elem(1k) - floor)/10) for where the element resistors'
    own thermal noise equals the digital floor. No derivative, no argmax,
    and snr_elem_db is monotone in R -- 137.60 dB at 1k falling to
    130.88 at 4.7k. Lower is always quieter and always costs current.
    There is nothing to be at an optimum of.
  * The figure is 0.67 dB, not 1.1. The 1.1 is the element resistors
    measured alone; through the stage it is 126.50 against 125.83.

Struck in place rather than quietly restated, in 0014 and in the module's
power page. What survives is that the one-unit-load rule really is
retired, so the value can be revisited for about 0.67 dB.

Three other corrections from the same pass. 0014 specified a 15 V TVS
where the board fits the 18 V part it was changed to. 0013 carried a
git-lfs row reading "missing" two rows below one reading "installed",
which its own correction claimed to have fixed. And parts-notes.md still
described U14 as sitting on the pump's 5.69 V output programmed to
4.99 V -- the exact paragraph that documented the fault -- now corrected
with the fault recorded as a quotation beside it.

The freshness checker's worst hole is closed, and it was mine:
SUPERSEDED_OK exempted docs/decisions/ wholesale, so the only content
che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
Other:
- title: The bipolar rail (decision 5, option B; supersedes 0009's -> The bipolar rail (0015, superseding 0009's
Changed lines of the file:
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@@
 	(generator "lyrebird")
 	(paper "User" 178 249)
-	(title_block (title "The bipolar rail (decision 5, option B; supersedes 0009's"))
+	(title_block (title "The bipolar rail (0015, superseding 0009's"))
 	(symbol (lib_id "Device:C") (at 35.56 35.56 0) (unit 1)
 		(exclude_from_sim no) (in_bom yes) (on_board yes) (dnp no)

Commit message: Act on the schematic validation: three faults and the core-rail guard
**The SuperSpeed pairs were wired backwards, and are now not wired.**
USB_SSRX_P/N were the only multi-node nets on the board with an INPUT at
every pin -- the receptacle's SSRX pins are inputs and so are the
bridge's RIDP/RIDN, so nothing drove them, and the transmit pair was
mirrored the same way. The comment asserted a crossover inside the cable
as fact and reasoned from it; USB 3.0 cables have no crossover.
SuperSpeed would never have trained and the link would have fallen back
to 480 Mb/s silently -- which is the speed 0014 chose on purpose, since
no galvanic isolator exists above USB 2.0. So the pairs are removed
rather than corrected, which also retires the hardest constraint in this
board's layout. How to wire them correctly if they ever come back is
recorded where they were.

**The inverting converter had no input capacitor across its own
terminals.** Nothing spanned +12V and -6V_A, and U7's GND pin *is*
-6V_A, so the loop its switching current actually takes was unbypassed
-- the input caps near U5 are referenced to system ground and are not in
that loop at all. This is the third fault found in U7 and all three are
the same mistake: reasoning about it as though its ground were the
board's.

**The translator's output enables are tied low against an explicit
datasheet instruction**, and the fix is sequencing rather than a pull-up.
SCES576I says OE must be pulled up to VCCA and not enabled until both
supplies are stable; a pull-up is not available here because nothing on
the module could pull it down -- no spare mezzanine pin, and MUTE_N has
the wrong polarity. Instead VCC(A) is made the last rail to arrive:
10 uF on U9's SET gives 573 ms against 359 ms for VCC(B), so the enable
cannot precede the supply it switches to. It costs nothing, because that
rail feeds the translator's reference supply and nothing else.

**The core rail now has a guard, and it needed two attempts.** The
existing as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
Parts:
- R10: value 45.3k 0.1% -> 40.2k 0.1%
- U14: value LT3045 op amp positive rail, +4.53 V from mezzanine 5 V -> LT3045 op amp positive rail, +4.02 V from mezzanine 5 V
Changed lines of the file:
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@@
 		(property "Reference" "R10" (at 86.36 114.15 0)
 			(effects (font (size 1.27 1.27))))
-		(property "Value" "45.3k 0.1%" (at 86.36 134.77 0)
+		(property "Value" "40.2k 0.1%" (at 86.36 134.77 0)
 			(effects (font (size 1.27 1.27))))
 		(instances (project "" (path "/" (reference "R10") (unit 1))))
@@
 		(property "Reference" "U14" (at 45.72 149.71 0)
 			(effects (font (size 1.27 1.27))))
-		(property "Value" "LT3045 op amp positive rail, +4.53 V from mezzanine 5 V" (at 45.72 175.41 0)
+		(property "Value" "LT3045 op amp positive rail, +4.02 V from mezzanine 5 V" (at 45.72 175.41 0)
 			(effects (font (size 1.27 1.27))))
 		(instances (project "" (path "/" (reference "U14") (unit 1))))
