File: hardware/lyrebird-dac-reva/sheets/05-Precision-rails-The-element-reference-sets-full-.kicad_sch (KiCad schematic)
At the start: 9 parts, among them U5 LT3045 element reference, U6 LT3045 clock chain, U9 LT3045 header-side 2.5 V

Commit message: Act on the schematic validation: three faults and the core-rail guard
**The SuperSpeed pairs were wired backwards, and are now not wired.**
USB_SSRX_P/N were the only multi-node nets on the board with an INPUT at
every pin -- the receptacle's SSRX pins are inputs and so are the
bridge's RIDP/RIDN, so nothing drove them, and the transmit pair was
mirrored the same way. The comment asserted a crossover inside the cable
as fact and reasoned from it; USB 3.0 cables have no crossover.
SuperSpeed would never have trained and the link would have fallen back
to 480 Mb/s silently -- which is the speed 0014 chose on purpose, since
no galvanic isolator exists above USB 2.0. So the pairs are removed
rather than corrected, which also retires the hardest constraint in this
board's layout. How to wire them correctly if they ever come back is
recorded where they were.

**The inverting converter had no input capacitor across its own
terminals.** Nothing spanned +12V and -6V_A, and U7's GND pin *is*
-6V_A, so the loop its switching current actually takes was unbypassed
-- the input caps near U5 are referenced to system ground and are not in
that loop at all. This is the third fault found in U7 and all three are
the same mistake: reasoning about it as though its ground were the
board's.

**The translator's output enables are tied low against an explicit
datasheet instruction**, and the fix is sequencing rather than a pull-up.
SCES576I says OE must be pulled up to VCCA and not enabled until both
supplies are stable; a pull-up is not available here because nothing on
the module could pull it down -- no spare mezzanine pin, and MUTE_N has
the wrong polarity. Instead VCC(A) is made the last rail to arrive:
10 uF on U9's SET gives 573 ms against 359 ms for VCC(B), so the enable
cannot precede the supply it switches to. It costs nothing, because that
rail feeds the translator's reference supply and nothing else.

**The core rail now has a guard, and it needed two attempts.** The
existing as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
Parts:
- C35: value 4.7uF -> 10uF
Changed lines of the file:
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@@
 		(property "Reference" "C35" (at 45.72 197.97 0)
 			(effects (font (size 1.27 1.27))))
-		(property "Value" "4.7uF" (at 45.72 218.59 0)
+		(property "Value" "10uF" (at 45.72 218.59 0)
 			(effects (font (size 1.27 1.27))))
 		(instances (project "" (path "/" (reference "C35") (unit 1))))
