File: hardware/lyrebird-dac-reva/sheets/01-Element-resistors-Thin-film-arrays-so-elements-s.kicad_sch (KiCad schematic)
At the start: 42 parts

Commit message: Work the reconciliation's top five, and stop checks passing on nothing
Four of the five are done and the fifth cannot be done from a PDF.

The abs-max allowance is per pin, the core check covers the bridge as
well as the FPGA and walks bridges of any pin count, and interface.md no
longer claims the oscillator rule is enforced. What remained from that
list is here.

**Checks now assert they found something.** This project has now been
bitten three times by a check reporting success because it located no
subjects: a netlist reader looking for pin-name fields the netlist does
not contain, assert_core_rail with its pin names matching nothing, and
ldo_rails failing open three ways -- a value spelled 40200R rather than
40.2k, an IN rail missing from a small map, or a family name absent from
a component value, each silently dropping a regulator. So
verify_power.py asserts six post-regulators, assert_core_rail fails when
it finds no core pins, and assert_below_abs_max fails when given nothing
to protect. All three tamper-tested. The 40200R tamper now fails where
it used to pass 17 of 17.

**The element split is even**, 1.65k twice rather than 1.69k + 1.65k.
The asymmetry existed because 3.30 kohm is below the 3312 ohm the
one-unit-load rule demanded at power-on, and 0014 retired that rule. An
even split is better on everything that survives: slightly quieter,
both halves of every element matched by construction rather than by
tolerance, and one BOM line instead of two. The pole moves 1.059 to
1.072 MHz, three decades above the band.

**main-reva/power.md's "What has no source today" is gone**, and it is
worth saying what it said: that the LTM4622 was absent so the 1.0 V and
2.5 V rails had no regulator, that there was no USB connector so the
5 V input had no entry point, and that the VBUS ferrite was missing.
Five sentences, four of them false, about the rails that power the FPGA.
All true when written and none since. Replaced with a table of what
actually sources each rail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
Parts:
- RN1, RN2, RN3, RN4, RN5, RN6, RN7: value 1.69k 0.1% thin film -> 1.65k 0.1% thin film
Changed lines of the file:
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@@
 		(property "Reference" "RN2" (at 68.58 59.540000000000006 0)
 			(effects (font (size 1.27 1.27))))
-		(property "Value" "1.69k 0.1% thin film" (at 68.58 82.7 0)
+		(property "Value" "1.65k 0.1% thin film" (at 68.58 82.7 0)
 			(effects (font (size 1.27 1.27))))
 		(instances (project "" (path "/" (reference "RN2") (unit 1))))
@@
 		(property "Reference" "RN3" (at 226.06 59.540000000000006 0)
 			(effects (font (size 1.27 1.27))))
-		(property "Value" "1.69k 0.1% thin film" (at 226.06 82.7 0)
+		(property "Value" "1.65k 0.1% thin film" (at 226.06 82.7 0)
 			(effects (font (size 1.27 1.27))))
 		(instances (project "" (path "/" (reference "RN3") (unit 1))))
@@
 		(property "Reference" "RN4" (at 106.68 143.35999999999999 0)
 			(effects (font (size 1.27 1.27))))
-		(property "Value" "1.69k 0.1% thin film" (at 106.68 166.52 0)
+		(property "Value" "1.65k 0.1% thin film" (at 106.68 166.52 0)
 			(effects (font (size 1.27 1.27))))
 		(instances (project "" (path "/" (reference "RN4") (unit 1))))
@@
 		(property "Reference" "RN5" (at 226.06 143.35999999999999 0)
 			(effects (font (size 1.27 1.27))))
-		(property "Value" "1.69k 0.1% thin film" (at 226.06 166.52 0)
+		(property "Value" "1.65k 0.1% thin film" (at 226.06 166.52 0)
 			(effects (font (size 1.27 1.27))))
 		(instances (project "" (path "/" (reference "RN5") (unit 1))))
@@
 		(property "Reference" "RN6" (at 106.68 227.17999999999998 0)
 			(effects (font (size 1.27 1.27))))
-		(property "Value" "1.69k 0.1% thin film" (at 106.68 250.34 0)
+		(property "Value" "1.65k 0.1% thin film" (at 106.68 250.34 0)
 			(effects (font (size 1.27 1.27))))
 		(instances (project "" (path "/" (reference "RN6") (unit 1))))
@@
 		(property "Reference" "RN7" (at 226.06 227.17999999999998 0)
 			(effects (font (size 1.27 1.27))))
-		(property "Value" "1.69k 0.1% thin film" (at 226.06 250.34 0)
+		(property "Value" "1.65k 0.1% thin film" (at 226.06 250.34 0)
 			(effects (font (size 1.27 1.27))))
 		(instances (project "" (path "/" (reference "RN7") (unit 1))))
@@
 		(property "Reference" "RN1" (at 68.58 311.0 0)
 			(effects (font (size 1.27 1.27))))
-		(property "Value" "1.69k 0.1% thin film" (at 68.58 334.15999999999997 0)
+		(property "Value" "1.65k 0.1% thin film" (at 68.58 334.15999999999997 0)
 			(effects (font (size 1.27 1.27))))
 		(instances (project "" (path "/" (reference "RN1") (unit 1))))
